File: Circuito/Circuito.kicad_sch (KiCad schematic)
At the start: 4 parts, among them J6 Screw_Terminal_01x09, J7 Screw_Terminal_01x09, J8 Screw_Terminal_01x09, J9 Screw_Terminal_01x09

Commit message: commit
Parts:
- added D6: SMF24CA, PCM_Diode_SMD_AKL:D_SOD-123F, symbol Diode_TVS_AKL:SMF24CA
- J6, J7, J8, J9: footprint (none) -> TerminalBlock_Phoenix:TerminalBlock_Phoenix_PT-1,5-9-5.0-H_1x09_P5.00mm_Horizontal
Connections:
- net PLC/4_20mA_2_OUT is gone; now on net PLC/0_10V_1_OUT: J9.8 (Pin_8)
- net PLC/0_10V_1_OUT: no longer J9.9 (Pin_9)
- net PLC/AC_N: no longer J7.7 (Pin_7)
- net PLC/AC_P: now also J7.9 (Pin_9); no longer J7.6 (Pin_6)
- net PLC/CT_N: now also J7.6 (Pin_6); no longer J7.9 (Pin_9)
- net PLC/CT_P: now also J7.7 (Pin_7); no longer J7.8 (Pin_8)
- net +24V: now reaches J6.1 (Pin_1)
- net +24V: now also D6.2 (A)
- net GND: now reaches J6.2 (Pin_2)
- net GND: now also J9.9 (Pin_9), D6.1 (K)
- new net Earth: J7.8 (Pin_8)
Other:
- added sheet PowerSupply (PowerSupply.kicad_sch)
- sheet PLC ports: added none; removed 0-10V_2_OUT, 4_20mA_2_OUT
