File: Circuito/RLY.kicad_sch (KiCad schematic)
At the start: 0 parts

Commit message: commit
Parts:
- added K1, K2: G5V-1, Relay_THT:Relay_SPDT_Omron_G5V-1, symbol Relay:G5V-1
- added U13: LK1802, PCM_JLCPCB:SOT-23-6_L2.9-W1.6-P0.95-LS2.8-BR, symbol easyeda2kicad:LK1802
Connections:
- net RLY_1_COM: now also K1.5, K1.6
- net RLY_1_NC: now also K1.1
- net RLY_1_NO: now also K1.10
- net RLY_2_COM: now also K2.5, K2.6
- net RLY_2_NC: now also K2.1
- net RLY_2_NO: now also K2.10
- new net: K1.9, U13.6 (2C)
- new net: K2.9, U13.1 (1C)
- new net +24V: K1.2, K2.2, U13.5 (COM)
- new net DRV_RLY_1: U13.3 (1B)
- new net DRV_RLY_2: U13.4 (2B)
- new net GND: U13.2 (E)
