File: Circuito/4-20mA_OUT.kicad_sch (KiCad schematic)
At the start: 11 parts, among them Q4 NCE60P04R, U8 GP8302-TC50-EW

Commit message: Last commit
Parts:
- D15: footprint Diode_SMD_AKL:D_SMB -> PCM_Diode_SMD_AKL:D_SMB
- Q4: footprint EasyEDA:SOT-223-3_L6.5-W3.4-P2.30-LS7.0-BR -> PCM_JLCPCB:SOT-223-3_L6.5-W3.4-P2.30-LS7.0-BR
Changed lines of the file:
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@@
 			)
 		)
-		(property "Footprint" "EasyEDA:SOT-223-3_L6.5-W3.4-P2.30-LS7.0-BR"
+		(property "Footprint" "PCM_JLCPCB:SOT-223-3_L6.5-W3.4-P2.30-LS7.0-BR"
 			(at 182.88 83.82 0)
 			(effects
@@
 			)
 		)
-		(property "Footprint" "Diode_SMD_AKL:D_SMB"
+		(property "Footprint" "PCM_Diode_SMD_AKL:D_SMB"
 			(at 195.58 113.03 0)
 			(effects
