File: Circuito/EnergyMeterA1.kicad_sch (KiCad schematic)
At the start: 23 parts, among them U16 BL0942, U17 B0303S-1WR3_C7465185, U18 ISO7021DR

Commit message: Last commit
Parts:
- U18: footprint EasyEDA:SOIC-8_L4.9-W3.9-P1.27-LS6.0-BL -> PCM_JLCPCB:SOIC-8_L4.9-W3.9-P1.27-LS6.0-BL
Changed lines of the file:
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@@
 			)
 		)
-		(property "Footprint" "EasyEDA:SOIC-8_L4.9-W3.9-P1.27-LS6.0-BL"
+		(property "Footprint" "PCM_JLCPCB:SOIC-8_L4.9-W3.9-P1.27-LS6.0-BL"
 			(at 215.9 106.68 0)
 			(effects
