File: Circuito/NPN_IN.kicad_sch (KiCad schematic)
At the start: 6 parts, among them U2 AT3H4B-CUH-S

Commit message: Last commit
Parts:
- U2: footprint easyeda2kicad:SSOP-4_L2.7-W4.6-P1.27-LS7.0-TL -> EasyEDA:SSOP-4_L2.7-W4.6-P1.27-LS7.0-TL
Changed lines of the file:
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@@
 			)
 		)
-		(property "Footprint" "easyeda2kicad:SSOP-4_L2.7-W4.6-P1.27-LS7.0-TL"
+		(property "Footprint" "EasyEDA:SSOP-4_L2.7-W4.6-P1.27-LS7.0-TL"
 			(at 146.05 78.74 0)
 			(effects
