File: Circuito/OUT-PNP.kicad_sch (KiCad schematic)
At the start: 5 parts, among them U9 BTS723GWXUMA1

Commit message: Last commit
Parts:
- U9: footprint EasyEDA:SOIC-14_L8.7-W3.9-P1.27-LS6.0-BL -> PCM_JLCPCB:SOIC-14_L8.7-W3.9-P1.27-LS6.0-BL
Changed lines of the file:
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@@
 			)
 		)
-		(property "Footprint" "EasyEDA:SOIC-14_L8.7-W3.9-P1.27-LS6.0-BL"
+		(property "Footprint" "PCM_JLCPCB:SOIC-14_L8.7-W3.9-P1.27-LS6.0-BL"
 			(at 133.35 127 0)
 			(effects
