File: Circuito/PowerSupply.kicad_sch (KiCad schematic)
At the start: 6 parts, among them U3 PS-TO220

Commit message: Last commit
Parts:
- D3: footprint Snapeda:SMF3.3_SODFL3718X108N -> Diode_SMD:D_SOD-123
- U3: footprint MG_footprints:PS-TO-220-3_Vertical -> Package_TO_SOT_THT:TO-220-3_Vertical
Changed lines of the file:
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@@
 			)
 		)
-		(property "Footprint" "Snapeda:SMF3.3_SODFL3718X108N"
-			(at 215.9 82.55 0)
-			(effects
-				(font
-					(size 1.27 1.27)
-				)
-				(justify bottom)
-				(hide yes)
-			)
-		)
-		(property "Datasheet" ""
+		(property "Footprint" "Diode_SMD:D_SOD-123"
+			(at 215.9 82.55 0)
+			(effects
+				(font
+					(size 1.27 1.27)
+				)
+				(justify bottom)
+				(hide yes)
+			)
+		)
+		(property "Datasheet" "C2649858"
 			(at 215.9 82.55 0)
 			(effects
@@
 			)
 		)
-		(property "Footprint" "MG_footprints:PS-TO-220-3_Vertical"
+		(property "Footprint" "Package_TO_SOT_THT:TO-220-3_Vertical"
 			(at 172.72 69.215 0)
 			(effects
